Commit message: Add modified SO101 teleop tools

File: config/SO101/so101_new_calib.urdf (robot description, URDF)
Before this commit: robot so101_new_calib, 8 links, 7 joints
Joints:
- joint elbow_flex: origin xyz=-0.11257 -0.028 1.73763e-16 rpy=-3.63608e-16 8.74301e-16 1.5708 -> xyz=-0.1880 -0.028 1.73763e-16 rpy=-3.63608e-16 8.74301e-16 1.5708
- joint wrist_flex: origin xyz=-0.1349 0.0052 3.62355e-17 rpy=4.02456e-15 8.67362e-16 -1.5708 -> xyz=-0.2300 0.0052 3.62355e-17 rpy=4.02456e-15 8.67362e-16 -1.5708
